Commit message: week 2 tasks again attempted

File: src/humanoid_description/urdf/humanoid.urdf.xacro (robot description, xacro)
@@ -1,159 +1,84 @@
 <?xml version="1.0"?>
-  <robot name="humanoid" xmlns:xacro="http://www.ros.org/wiki/xacro">
-    <!-- Properties -->
-    <xacro:property name="PI" value="3.1415926535897931" />
-    <xacro:property name="DEG_TO_RAD" value="${PI/180}" />
-    <xacro:property name="TORSO_HEIGHT" value="0.8" />
-    <xacro:property name="TORSO_WIDTH" value="0.3" />
-    <xacro:property name="TORSO_LENGTH" value="0.4" />
-    <xacro:property name="SHOULDER_SIZE" value="0.4" />
-    <xacro:property name="HEAD_RADIUS" value="0.3" />
-    <xacro:property name="EYE_RADIUS" value="0.05" />
-    <xacro:property name="EYE_POS_X" value="0.08" /> <!-- X-offset from head center -->
-    <xacro:property name="EYE_POS_Y" value="${HEAD_RADIUS - 0.01}" /> <!-- Y-offset from head center (slightly protruding) -->
-    <xacro:property name="EYE_POS_Z" value="0.05" /> <!-- Z-offset from head center -->
-    <!-- Materials -->
-    <material name="blue">
-      <color rgba="0 0 0.8 1"/>
-    </material>
-    <material name="red">
-      <color rgba="0.8 0 0 1"/>
-    </material>
-    <material name="green">
-      <color rgba="0 0.8 0 1"/>
-    </material>
-    <material name="white">
-      <color rgba="1 1 1 1"/>
-    </material>
-    <!-- Base Link -->
-    <link name="base_link">
-      <visual>
-        <geometry><box size="0.01 0.01 0.01"/></geometry>
-        <material name="green"/>
-      </visual>
+<robot xmlns:xacro="http://www.ros.org/wiki/xacro" name="humanoid">
+    <xacro:property name="torso_color" value="0.2 0.5 1.0 1.0"/> <xacro:property name="head_color" value="1.0 0.2 0.2 1.0"/> <xacro:property name="eye_color" value="0 0 0 1.0"/>      <xacro:property name="camera_color" value="0.1 0.1 0.1 1.0"/> <link name="torso_link">
+        <visual>
+            <geometry><box size="0.4 0.3 0.6"/></geometry>
+            <material name="blue"><color rgba="${torso_color}"/></material>
+        </visual>
+        <collision><geometry><box size="0.4 0.3 0.6"/></geometry></collision>
+        <inertial>
+            <mass value="10"/>
+            <inertia ixx="1.0" ixy="0.0" ixz="0.0" iyy="1.0" iyz="0.0" izz="1.0"/>
+        </inertial>
     </link>
-    <!-- TORSO LINK -->
-    <joint name="base_to_torso_joint" type="fixed">
-      <parent link="base_link"/>
-      <child link="torso_link"/>
-      <origin xyz="0 0 ${TORSO_HEIGHT/2}" rpy="0 0 0"/>
-    </joint>
-    <link name="torso_link">
-      <visual>
-        <geometry><box size="${TORSO_WIDTH} ${TORSO_LENGTH} ${TORSO_HEIGHT}"/></geometry>
-        <material name="blue"/>
-      </visual>
-      <collision>
-        <geometry><box size="${TORSO_WIDTH} ${TORSO_LENGTH} ${TORSO_HEIGHT}"/></geometry>
-      </collision>
-      <inertial>
-        <origin xyz="0 0 0" rpy="0 0 0"/>
-        <mass value="20.0"/>
-        <inertia ixx="1.0" ixy="0.0" ixz="0.0" iyy="1.0" iyz="0.0" izz="1.0"/>
-      </inertial>
+    <link name="head_link">
+        <visual>
+            <geometry><sphere radius="0.15"/></geometry>
+            <material name="red"><color rgba="${head_color}"/></material>
+        </visual>
+        <collision><geometry><sphere radius="0.15"/></geometry></collision>
+        <inertial>
+            <mass value="2"/>
+            <inertia ixx="0.1" ixy="0.0" ixz="0.0" iyy="0.1" iyz="0.0" izz="0.1"/>
+        </inertial>
     </link>
-    <!-- RIGHT SHOULDER LINK -->
-    <joint name="torso_to_right_shoulder_joint" type="fixed">
-      <parent link="torso_link"/>
-      <child link="right_shoulder_link"/>
-      <origin xyz="${TORSO_WIDTH/2 + SHOULDER_SIZE/2 - 0.1} 0 ${TORSO_HEIGHT/2 + SHOULDER_SIZE/2 - 0.4}" rpy="0 0 0"/>
-    </joint>
-    <link name="right_shoulder_link">
-      <visual>
-        <geometry><box size="0.2 ${SHOULDER_SIZE} ${SHOULDER_SIZE}"/></geometry>
-        <material name="green"/>
-      </visual>
-      <collision>
-        <geometry><box size="0.2 ${SHOULDER_SIZE} ${SHOULDER_SIZE}"/></geometry>
-      </collision>
-      <inertial>
-        <origin xyz="0 0 0" rpy="0 0 0"/>
-        <mass value="2.0"/>
-        <inertia ixx="0.1" ixy="0.0" ixz="0.0" iyy="0.1" iyz="0.0" izz="0.1"/>
-      </inertial>
-    </link>
-    <!-- LEFT SHOULDER LINK -->
-    <joint name="torso_to_left_shoulder_joint" type="fixed">
-      <parent link="torso_link"/>
-      <child link="left_shoulder_link"/>
-      <origin xyz="-${TORSO_WIDTH/2 + SHOULDER_SIZE/2 - 0.1} 0 ${TORSO_HEIGHT/2 + SHOULDER_SIZE/2 -0.4}" rpy="0 0 0"/>
-    </joint>
-    <link name="left_shoulder_link">
-      <visual>
-        <geometry><box size="0.2 ${SHOULDER_SIZE} ${SHOULDER_SIZE}"/></geometry>
-        <material name="green"/>
-      </visual>
-      <collision>
-        <geometry><box size="0.2 ${SHOULDER_SIZE} ${SHOULDER_SIZE}"/></geometry>
-      </collision>
-      <inertial>
-        <origin xyz="0 0 0" rpy="0 0 0"/>
-        <mass value="2.0"/>
-        <inertia ixx="0.1" ixy="0.0" ixz="0.0" iyy="0.1" iyz="0.0" izz="0.1"/>
-      </inertial>
-    </link>
-    <!-- NECK JOINT (Head rotation) -->
     <joint name="neck_joint" type="revolute">
-      <parent link="torso_link"/>
-      <child link="head_link"/>
-      <origin xyz="0 0 ${TORSO_HEIGHT/2 + HEAD_RADIUS}" rpy="0 0 0"/>
-      <axis xyz="0 0 1"/>
-      <limit lower="-${90 * DEG_TO_RAD}" upper="${90 * DEG_TO_RAD}"
-             effort="100" velocity="10"/>
-    </joint>
-    <!-- HEAD LINK -->
-    <link name="head_link">
-      <visual>
-        <geometry><sphere radius="${HEAD_RADIUS}"/></geometry>
-        <material name="red"/>
-      </visual>
-      <collision>
-        <geometry><sphere radius="${HEAD_RADIUS}"/></geometry>
-      </collision>
-      <inertial>
-        <origin xyz="0 0 0" rpy="0 0 0"/>
-        <mass value="5.0"/>
-        <inertia ixx="0.2" ixy="0.0" ixz="0.0" iyy="0.2" iyz="0.0" izz="0.2"/>
-      </inertial>
-    </link>
-    <!-- RIGHT EYE LINK -->
-    <joint name="head_to_right_eye_joint" type="fixed">
-      <parent link="head_link"/>
-      <child link="right_eye_link"/>
-      <origin xyz="${EYE_POS_X} ${EYE_POS_Y} ${EYE_POS_Z}" rpy="0 0 0"/>
-    </joint>
-    <link name="right_eye_link">
-      <visual>
-        <geometry><sphere radius="${EYE_RADIUS}"/></geometry>
-        <material name="white"/>
-      </visual>
-      <collision>
-        <geometry><sphere radius="${EYE_RADIUS}"/></geometry>
-      </collision>
-      <inertial>
-        <origin xyz="0 0 0" rpy="0 0 0"/>
-        <mass value="0.1"/>
-        <inertia ixx="0.001" ixy="0.0" ixz="0.0" iyy="0.001" iyz="0.0" izz="0.001"/>
-      </inertial>
-    </link>
-    <!-- LEFT EYE LINK -->
-    <joint name="head_to_left_eye_joint" type="fixed">
-      <parent link="head_link"/>
-      <child link="left_eye_link"/>
-      <origin xyz="-${EYE_POS_X} ${EYE_POS_Y} ${EYE_POS_Z}" rpy="0 0 0"/>
+        <parent link="torso_link"/>
+        <child link="head_link"/>
+        <origin xyz="0 0 0.4" rpy="0 0 0"/>
+        <axis xyz="0 0 1"/>
+        <limit lower="-1.57" upper="1.57" effort="10" velocity="1.0"/>
     </joint>
     <link name="left_eye_link">
+        <visual><geometry><sphere radius="0.02"/></geometry><material name="black"><color rgba="${eye_color}"/></material></visual>
+    </link>
+    <link name="right_eye_link">
+        <visual><geometry><sphere radius="0.02"/></geometry><material name="black"><color rgba="${eye_color}"/></material></visual>
+    </link>
+    <joint name="left_eye_joint" type="fixed">
+        <parent link="head_link"/><child link="left_eye_link"/><origin xyz="0.14 0.05 0.05" rpy="0 0 0"/>
+    </joint>
+    <joint name="right_eye_joint" type="fixed">
+        <parent link="head_link"/><child link="right_eye_link"/><origin xyz="0.14 -0.05 0.05" rpy="0 0 0"/>
+    </joint>
+    <link name="camera_link">
       <visual>
-        <geometry><sphere radius="${EYE_RADIUS}"/></geometry>
-        <material name="white"/>
+        <geometry><box size="0.05 0.05 0.05"/></geometry>
+        <material name="camera_mat"><color rgba="${camera_color}"/></material>
       </visual>
-      <collision>
-        <geometry><sphere radius="${EYE_RADIUS}"/></geometry>
-      </collision>
-      <inertial>
-        <origin xyz="0 0 0" rpy="0 0 0"/>
-        <mass value="0.1"/>
-        <inertia ixx="0.001" ixy="0.0" ixz="0.0" iyy="0.001" iyz="0.0" izz="0.001"/>
-      </inertial>
+      <collision><geometry><box size="0.05 0.05 0.05"/></geometry></collision>
+      <inertial><mass value="0.01"/><inertia ixx="1e-6" ixy="0" ixz="0" iyy="1e-6" iyz="0" izz="1e-6" /></inertial>
     </link>
-  </robot>
+    <joint name="camera_joint" type="fixed">
+      <parent link="head_link"/>
+      <child link="camera_link"/>
+      <origin xyz="0.12 0 0" rpy="0 0 0"/>
+    </joint>
+    <gazebo reference="torso_link">
+        <sensor name="imu_sensor" type="imu">
+            <plugin name="gazebo_ros_imu_sensor" filename="libgazebo_ros_imu_sensor.so">
+                <ros>
+                    <namespace>/humanoid</namespace>
+                    <remapping>~/out:=imu_data</remapping>
+                </ros>
+            </plugin>
+        </sensor>
+    </gazebo>
+    <gazebo reference="camera_link">
+        <sensor name="camera_sensor" type="camera">
+            <update_rate>30.0</update_rate>
+            <camera name="head_camera">
+                <horizontal_fov>1.396</horizontal_fov>
+                <image><width>800</width><height>800</height><format>R8G8B8</format></image>
+                <clip><near>0.02</near><far>300</far></clip>
+            </camera>
+            <plugin name="camera_controller" filename="libgazebo_ros_camera.so">
+                <ros>
+                    <namespace>/humanoid</namespace>
+                    <remapping>~/image_raw:=image_raw</remapping>
+                    <remapping>~/camera_info:=camera_info</remapping>
+                </ros>
+            </plugin>
+        </sensor>
+    </gazebo>
+</robot>

Commit message: Added trigger system and movement

File: src/humanoid_description/urdf/humanoid.urdf.xacro (robot description, xacro)
@@ -1,5 +1,11 @@
 <?xml version="1.0"?>
 <robot xmlns:xacro="http://www.ros.org/wiki/xacro" name="humanoid">
-    <xacro:property name="torso_color" value="0.2 0.5 1.0 1.0"/> <xacro:property name="head_color" value="1.0 0.2 0.2 1.0"/> <xacro:property name="eye_color" value="0 0 0 1.0"/>      <xacro:property name="camera_color" value="0.1 0.1 0.1 1.0"/> <link name="torso_link">
+    <!-- Color Properties -->
+    <xacro:property name="torso_color" value="0.2 0.5 1.0 1.0"/>
+    <xacro:property name="head_color" value="1.0 0.2 0.2 1.0"/>
+    <xacro:property name="eye_color" value="0 0 0 1.0"/>
+    <xacro:property name="camera_color" value="0.1 0.1 0.1 1.0"/>
+    <!-- Main Body Links and Joints -->
+    <link name="torso_link">
         <visual>
             <geometry><box size="0.4 0.3 0.6"/></geometry>
@@ -12,4 +18,8 @@
         </inertial>
     </link>
+    <!-- Gazebo color tag for the torso -->
+    <gazebo reference="torso_link">
+        <material>Gazebo/Blue</material>
+    </gazebo>
     <link name="head_link">
         <visual>
@@ -23,4 +33,8 @@
         </inertial>
     </link>
+    <!-- Gazebo color tag for the head -->
+    <gazebo reference="head_link">
+        <material>Gazebo/Red</material>
+    </gazebo>
     <joint name="neck_joint" type="revolute">
         <parent link="torso_link"/>
@@ -33,7 +47,15 @@
         <visual><geometry><sphere radius="0.02"/></geometry><material name="black"><color rgba="${eye_color}"/></material></visual>
     </link>
+    <!-- Gazebo color tag for the left eye -->
+    <gazebo reference="left_eye_link">
+        <material>Gazebo/Black</material>
+    </gazebo>
     <link name="right_eye_link">
         <visual><geometry><sphere radius="0.02"/></geometry><material name="black"><color rgba="${eye_color}"/></material></visual>
     </link>
+    <!-- Gazebo color tag for the right eye -->
+    <gazebo reference="right_eye_link">
+        <material>Gazebo/Black</material>
+    </gazebo>
     <joint name="left_eye_joint" type="fixed">
         <parent link="head_link"/><child link="left_eye_link"/><origin xyz="0.14 0.05 0.05" rpy="0 0 0"/>
@@ -50,4 +72,8 @@
       <inertial><mass value="0.01"/><inertia ixx="1e-6" ixy="0" ixz="0" iyy="1e-6" iyz="0" izz="1e-6" /></inertial>
     </link>
+    <!-- Gazebo color tag for the camera -->
+    <gazebo reference="camera_link">
+        <material>Gazebo/DarkGrey</material>
+    </gazebo>
     <joint name="camera_joint" type="fixed">
       <parent link="head_link"/>
@@ -55,4 +81,5 @@
       <origin xyz="0.12 0 0" rpy="0 0 0"/>
     </joint>
+    <!-- Sensor Plugins -->
     <gazebo reference="torso_link">
         <sensor name="imu_sensor" type="imu">
